File: PCB/gamepad.kicad_pcb (KiCad board)
At the start: 2 copper layers, 65 x 92.5 mm, 9 parts, among them J1 Conn_01x04, SW1 SW_Push, SW2 SW_Push, SW3 SW_Push, SW4 SW_Push, SW5 SW_Push, SW6 SW_Push, U1 XIAO-RP2040-DIP

Commit message: turn oled
Parts:
- moved J1 14.3 mm to (136.5, 54.3), turned to 180 degrees
Routing:
- net SDA: track 106.1 -> 85.1 mm
- net +5V: track 109.7 -> 121.3 mm
- net GND: track 193.7 -> 185.0 mm
- net SCL: track 78.1 -> 83.8 mm
